Commit message: Update parameters for real UR5e.

File: robo_manip_aug/assets/mujoco_ur5e/mujoco_ur5e.urdf (robot description, URDF)
Before this commit: robot mujoco_ur5e, 49 links, 48 joints
Joints:
- joint world2ur5e_root_frame_fixed: origin xyz=-0.605 0.0 0.8 rpy=0.0 0.0 0.0 -> xyz=0.0 0.0 0.0 rpy=0.0 0.0 0.0

Commit message: [assets] Attach a Hand-E gripper to the URDF model.

File: robo_manip_aug/assets/mujoco_ur5e/mujoco_ur5e.urdf (robot description, URDF)
Before this commit: robot mujoco_ur5e, 49 links, 48 joints
Links:
- removed link base_mount
- removed link base_mount2gripper_base_fixed_jointbody
- removed link gripper_base
- removed link left_coupler
- removed link left_coupler_joint_jointbody
- removed link left_driver
- removed link left_driver_joint_jointbody
- removed link left_follower
- removed link left_follower2left_pad_fixed_jointbody
- removed link left_follower_joint_jointbody
- removed link left_pad
- removed link left_pad2left_silicone_pad_fixed_jointbody
- removed link left_silicone_pad
- removed link left_spring_link
- removed link left_spring_link_joint_jointbody
- removed link right_coupler
- removed link right_coupler_joint_jointbody
- removed link right_driver
- removed link right_driver_joint_jointbody
- removed link right_follower
- removed link right_follower2right_pad_fixed_jointbody
- removed link right_follower_joint_jointbody
- removed link right_pad
- removed link right_pad2right_silicone_pad_fixed_jointbody
- removed link right_silicone_pad
- removed link right_spring_link
- removed link right_spring_link_joint_jointbody
- removed link wrist_3_link2base_mount_fixed_jointbody
- added link robotiq_hande_coupler, mass 0.119; collision cylinder length=0.0169 radius=0.0385; visual mesh filename=meshes/io_coupler.dae
- added link robotiq_hande_end
- added link robotiq_hande_left_finger, mass 0.03804; collision mesh filename=meshes/finger_collision.dae scale=1.0 1.0 1.0; visual mesh filename=meshes/finger.dae scale=1.0 1.0 1.0
- added link robotiq_hande_link, mass 0.86387; collision cylinder length=0.10690000000000001 radius=0.0385; visual mesh filename=meshes/hande.dae scale=1.0 1.0 1.0
- added link robotiq_hande_right_finger, mass 0.03804; collision mesh filename=meshes/finger_collision.dae scale=1.0 1.0 1.0; visual mesh filename=meshes/finger.dae scale=1.0 1.0 1.0
Joints:
- removed joint base_mount2gripper_base_fixed
- removed joint base_mount2gripper_base_fixed_offset
- removed joint left_coupler_joint
- removed joint left_coupler_joint_offset
- removed joint left_driver_joint
- removed joint left_driver_joint_offset
- removed joint left_follower2left_pad_fixed
- removed joint left_follower2left_pad_fixed_offset
- removed joint left_follower_joint
- removed joint left_follower_joint_offset
- removed joint left_pad2left_silicone_pad_fixed
- removed joint left_pad2left_silicone_pad_fixed_offset
- removed joint left_spring_link_joint
- removed joint left_spring_link_joint_offset
- removed joint right_coupler_joint
- removed joint right_coupler_joint_offset
- removed joint right_driver_joint
- removed joint right_driver_joint_offset
- removed joint right_follower2right_pad_fixed
- removed joint right_follower2right_pad_fixed_offset
- removed joint right_follower_joint
- removed joint right_follower_joint_offset
- removed joint right_pad2right_silicone_pad_fixed
- removed joint right_pad2right_silicone_pad_fixed_offset
- removed joint right_spring_link_joint
- removed joint right_spring_link_joint_offset
- removed joint wrist_3_link2base_mount_fixed
- removed joint wrist_3_link2base_mount_fixed_offset
- added joint robotiq_hande_base_joint: type fixed, parent robotiq_hande_coupler, child robotiq_hande_link, origin xyz=0 0 0.011 rpy=0 0 0
- added joint robotiq_hande_coupler_joint: type fixed, parent wrist_3_link, child robotiq_hande_coupler, origin xyz=0.0 0.1 0.0 rpy=-1.5707963267948957 0.0 0.0
- added joint robotiq_hande_end_joint: type fixed, parent robotiq_hande_link, child robotiq_hande_end, origin xyz=0 0 0.14550000000000002 rpy=0 0 0
- added joint robotiq_hande_left_finger_joint: type prismatic, parent robotiq_hande_link, child robotiq_hande_left_finger, origin xyz=0 0 0.099 rpy=0 0 0, axis 1 0 0, limit lower=0 upper=0.025 effort=130 velocity=0.15
- added joint robotiq_hande_right_finger_joint: type prismatic, parent robotiq_hande_link, child robotiq_hande_right_finger, origin xyz=0 0 0.099 rpy=0 0 0, axis -1 0 0, limit lower=0 upper=0.025 effort=130 velocity=0.15, mimic joint=robotiq_hande_left_finger_joint multiplier=1 offset=0
- joint wrist_3_link2d435i_fixed: origin xyz=0.0 0.1 -0.05 rpy=-1.5708000000000002 0.0 0.0 -> xyz=0.0 0.13 0.05 rpy=-1.5708000000000002 0.0 0.0
